File: PCB/servo.kicad_pcb (KiCad board)
At the start: 2 copper layers, 19 x 19 mm, 17 parts, among them J1 Conn_ARM_SWD_TagConnect_TC203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, J2 Conn_01x04_MountingPin, U1 ATSAMD21E17D-M, U2 TMC6300-LA-T, U3 MA730, U4 LDK130PU33R_DFN6

Commit message: Commit currrent work
Parts:
- added J3: Conn_01x06_MountingPin, Connector_JST:JST_SH_SM06B-SRSS-TB_1x06-1MP_P1.00mm_Horizontal, F.Cu at (50.0, 30.0)
- added J4: Conn_01x06_MountingPin, Connector_JST:JST_SH_SM06B-SRSS-TB_1x06-1MP_P1.00mm_Horizontal, F.Cu at (50.0, 38.8)
- added J5: XKB-USB-C16PIN, common:XKB-USB-C-16P, F.Cu at (41.3, 20.8)
- added R2: 5.1k, common:R_0402_1005Metric, F.Cu at (44.2, 22.5)
- added R3: 5.1k, common:R_0402_1005Metric, F.Cu at (44.2, 18.8)
- added U5: USBLC6-2P6, common:SOT-666, F.Cu at (45.5, 20.8)
- moved J1 30.9 mm to (55.1, 20.5), turned to 90 degrees
- moved TP3 25.2 mm to (49.0, 45.8)
- moved C7 22.4 mm to (45.2, 45.8), turned to 180 degrees
- moved U4 21.8 mm to (56.1, 50.1), turned to 90 degrees
- moved TP1 21.2 mm to (47.2, 43.5)
- moved C6 20.0 mm to (45.3, 47.0)
- moved TP2 18.1 mm to (43.0, 46.0)
- moved R1 15.7 mm to (54.5, 53.5), turned to 180 degrees
- moved C1 12.6 mm to (54.5, 56.2), turned to 180 degrees
- moved C3 12.4 mm to (56.1, 48.6), turned to 180 degrees
- moved C2 11.9 mm to (54.5, 55.0)
- moved C4 11.8 mm to (56.1, 51.6), turned to 180 degrees
- turned U3 to 90 degrees
Connections:
- U2 pad 16: unconnected-(U2-BRUV-Pad16) -> GND
- U2 pad 20: unconnected-(U2-BRW-Pad20) -> GND

Commit message: Update pcb
Parts:
- moved C5 0.25 mm to (47.0, 49.8)
Routing:
- net GND: track 0.00 -> 10.1 mm, vias 0 -> 5
- net /CLK: track 0.00 -> 8.27 mm
- net /VIO: track 0.00 -> 5.04 mm
- net /MOSI: track 0.00 -> 2.53 mm
- net Net-(U2-1.8VOUT): track 0.00 -> 1.60 mm
- net Net-(U2-W): track 0.00 -> 1.55 mm
- net +3.3V: track 0.00 -> 1.07 mm, vias 0 -> 1
Other:
- board size 19 x 19 mm -> 19 x 26 mm
- copper layers 2 -> 4

Commit message: Commit current PCB progress
Parts:
- moved TP1 2.36 mm to (48.1, 45.7)
- moved TP3 1.73 mm to (50.6, 46.4)
- moved J2 0.87 mm to (50.0, 61.1)
- moved J4 0.75 mm to (50.0, 39.5)
- moved TP2 0.68 mm to (42.6, 46.5)
- moved U1 0.65 mm to (50.0, 55.4)
- moved C6 0.40 mm to (44.9, 46.8)
- moved C7 0.40 mm to (44.9, 45.5)
- moved C3 0.08 mm to (56.1, 48.5)
Routing:
- net +5V: track 0.00 -> 63.9 mm, vias 0 -> 17
- net GND: track 10.1 -> 61.3 mm, vias 5 -> 33
- net D-: track 0.00 -> 30.6 mm, vias 0 -> 2
- net D+: track 0.00 -> 26.9 mm, vias 0 -> 2
- net SWDIO: track 0.00 -> 24.8 mm, vias 0 -> 2
- net SWCLK: track 0.00 -> 23.8 mm, vias 0 -> 2
- net +3.3V: track 1.07 -> 22.7 mm, vias 1 -> 3
- net /MISO: track 0.00 -> 14.2 mm, vias 0 -> 2
- net /WH: track 0.00 -> 12.8 mm
- net /CS: track 0.00 -> 10.6 mm, vias 0 -> 2
- net /UH: track 0.00 -> 9.85 mm, vias 0 -> 2
- net /VH: track 0.00 -> 9.51 mm, vias 0 -> 2
- net /WL: track 0.00 -> 9.48 mm
- net /UL: track 0.00 -> 8.41 mm, vias 0 -> 2
- net /VL: track 0.00 -> 8.32 mm
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- added copper zone on In2.Cu, net +5V
- added copper zone on B.Cu, net GND
- added copper zone on F.Cu, net GND
- added copper zone on In1.Cu, net GND
Other:
- board size 19 x 26 mm -> 24.5 x 48.2 mm
